File: kicad/rp2040_pmod.kicad_sch (KiCad schematic)
At the start: 27 parts, among them J1 Conn_02x06_Odd_Even, J2 USB_B_Micro, J3 Conn_01x03_Pin, SW1 SW_Push, U1 RP2040, U2 W25Q32JVZP, U3 TLV74333, Y1 12MHz

Commit message: generate gerbers bom and pos files
Parts:
- D1: value LED -> LED Red
- J1: LCSC (none) -> C2911299
- J2: JLCPCB Part # C132562 -> (none); LCSC (none) -> C132562
- SW1: JLCPCB Part # C115357 -> (none); LCSC (none) -> C115357
- U1: LCSC (none) -> C2040
- U2: JLCPCB Part # C2940197 -> (none); LCSC (none) -> C2940197
- U3: JLCPCB Part # C408972 -> (none); LCSC (none) -> C408972
- Y1: JLCPCB Part # C524716 -> (none); LCSC (none) -> C524716
Changed lines of the file:
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@@
       (effects (font (size 1.27 1.27)) hide)
     )
-    (property "JLCPCB Part #" "C2940197" (at 69.85 163.83 0)
+    (property "LCSC" "C2940197" (at 69.85 163.83 0)
       (effects (font (size 1.27 1.27)) hide)
     )
@@
       (effects (font (size 1.27 1.27)) hide)
     )
-    (property "JLCPCB Part #" "C524716" (at 77.47 101.6 90)
+    (property "LCSC" "C524716" (at 77.47 101.6 90)
       (effects (font (size 1.27 1.27)) hide)
     )
@@
     )
     (property "Datasheet" "~" (at 238.76 49.53 0)
+      (effects (font (size 1.27 1.27)) hide)
+    )
+    (property "LCSC" "C2911299" (at 238.76 49.53 0)
       (effects (font (size 1.27 1.27)) hide)
     )
@@
       (effects (font (size 1.27 1.27)) (justify right))
     )
-    (property "Value" "LED" (at 170.18 127.3175 90)
+    (property "Value" "LED Red" (at 170.18 127.3175 90)
       (effects (font (size 1.27 1.27)) (justify right))
     )
@@
       (effects (font (size 1.27 1.27)) hide)
     )
-    (property "JLCPCB Part #" "C132562" (at 49.53 58.42 0)
+    (property "LCSC" "C132562" (at 49.53 58.42 0)
       (effects (font (size 1.27 1.27)) hide)
     )
@@
       (effects (font (size 1.27 1.27)) hide)
     )
-    (property "JLCPCB Part #" "C115357" (at 36.83 146.05 0)
+    (property "LCSC" "C115357" (at 36.83 146.05 0)
       (effects (font (size 1.27 1.27)) hide)
     )
@@
       (effects (font (size 1.27 1.27)) hide)
     )
-    (property "JLCPCB Part #" "C408972" (at 229.87 85.09 0)
+    (property "LCSC" "C408972" (at 229.87 85.09 0)
       (effects (font (size 1.27 1.27)) hide)
     )
@@
       (effects (font (size 1.27 1.27)) hide)
     )
+    (property "LCSC" "C2040" (at 124.46 88.9 0)
+      (effects (font (size 1.27 1.27)) hide)
+    )
